File: Hardware/P1I1_DCPowerBus.kicad_sch (KiCad schematic)
At the start: 32 parts, among them IC3 RY8310, J1 Conn_01x04_Pin, J2 Conn_01x04_Pin, Q2 AO3401A, U1 MAX485

Commit message: add all
Parts:
- F2: footprint Fuse:Fuse_0402_1005Metric -> Fuse:Fuse_0603_1608Metric
- R14, R9: now not fitted
Connections:
- net GND: now also J2.1 (Pin_1); no longer J2.4 (Pin_4)
- net VCC: now also J2.4 (Pin_4); no longer J2.1 (Pin_1)
Changed lines of the file:
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@@
 	(wire
 		(pts
-			(xy 26.67 50.8) (xy 27.94 50.8)
-		)
-		(stroke
-			(width 0)
-			(type default)
-		)
-	)
-	(wire
-		(pts
 			(xy 121.92 21.59) (xy 123.19 21.59)
 		)
@@
 	(wire
 		(pts
-			(xy 30.48 55.88) (xy 26.67 55.88)
+			(xy 68.58 36.83) (xy 55.88 36.83)
 		)
 		(stroke
@@
 	(wire
 		(pts
-			(xy 68.58 36.83) (xy 55.88 36.83)
+			(xy 161.29 35.56) (xy 161.29 36.83)
 		)
 		(stroke
@@
 	(wire
 		(pts
-			(xy 161.29 35.56) (xy 161.29 36.83)
+			(xy 264.16 123.19) (xy 264.16 114.3)
 		)
 		(stroke
@@
 	(wire
 		(pts
-			(xy 264.16 123.19) (xy 264.16 114.3)
+			(xy 198.12 95.25) (xy 198.12 110.49)
 		)
 		(stroke
@@
 	(wire
 		(pts
-			(xy 198.12 95.25) (xy 198.12 110.49)
+			(xy 185.42 128.27) (xy 187.96 128.27)
 		)
 		(stroke
@@
 	(wire
 		(pts
-			(xy 185.42 128.27) (xy 187.96 128.27)
+			(xy 185.42 125.73) (xy 187.96 125.73)
 		)
 		(stroke
@@
 	(wire
 		(pts
-			(xy 185.42 125.73) (xy 187.96 125.73)
+			(xy 123.19 27.94) (xy 130.81 27.94)
 		)
 		(stroke
@@
 	(wire
 		(pts
-			(xy 123.19 27.94) (xy 130.81 27.94)
+			(xy 26.67 53.34) (xy 30.48 53.34)
 		)
 		(stroke
@@
 	(wire
 		(pts
-			(xy 30.48 53.34) (xy 26.67 53.34)
-		)
-		(stroke
-			(width 0)
-			(type default)
-		)
-	)
-	(wire
-		(pts
 			(xy 182.88 31.75) (xy 182.88 33.02)
 		)
@@
 	(wire
 		(pts
+			(xy 26.67 50.8) (xy 27.94 50.8)
+		)
+		(stroke
+			(width 0)
+			(type default)
+		)
+	)
+	(wire
+		(pts
 			(xy 267.97 123.19) (xy 264.16 123.19)
 		)
@@
 	(wire
 		(pts
-			(xy 27.94 50.8) (xy 27.94 49.53)
+			(xy 182.88 40.64) (xy 182.88 44.45)
 		)
 		(stroke
@@
 	(wire
 		(pts
-			(xy 182.88 40.64) (xy 182.88 44.45)
+			(xy 83.82 35.56) (xy 83.82 36.83)
 		)
 		(stroke
@@
 	(wire
 		(pts
-			(xy 83.82 35.56) (xy 83.82 36.83)
+			(xy 128.27 36.83) (xy 140.97 36.83)
 		)
 		(stroke
@@
 	(wire
 		(pts
-			(xy 128.27 36.83) (xy 140.97 36.83)
+			(xy 198.12 138.43) (xy 198.12 140.97)
 		)
 		(stroke
@@
 	(wire
 		(pts
-			(xy 198.12 138.43) (xy 198.12 140.97)
+			(xy 26.67 55.88) (xy 30.48 55.88)
+		)
+		(stroke
+			(width 0)
+			(type default)
+		)
+	)
+	(wire
+		(pts
+			(xy 27.94 50.8) (xy 27.94 49.53)
 		)
 		(stroke
@@
 	(global_label "B"
 		(shape input)
-		(at 30.48 53.34 0)
+		(at 30.48 55.88 0)
 		(fields_autoplaced yes)
 		(effects
@@
 		)
 		(property "Intersheetrefs" "${INTERSHEET_REFS}"
-			(at 34.7352 53.34 0)
+			(at 34.7352 55.88 0)
 			(effects
 				(font
@@
 	(global_label "A"
 		(shape input)
-		(at 30.48 55.88 0)
+		(at 30.48 53.34 0)
 		(fields_autoplaced yes)
 		(effects
@@
 		)
 		(property "Intersheetrefs" "${INTERSHEET_REFS}"
-			(at 34.5538 55.88 0)
+			(at 34.5538 53.34 0)
 			(effects
 				(font
@@
 			)
 		)
-		(property "Footprint" "Fuse:Fuse_0402_1005Metric"
+		(property "Footprint" "Fuse:Fuse_0603_1608Metric"
 			(at 40.64 29.718 90)
 			(effects
@@
 		(in_bom yes)
 		(on_board yes)
-		(dnp no)
+		(dnp yes)
 		(property "Reference" "R9"
 			(at 180.848 38.862 90)
@@
 	(symbol
 		(lib_id "Connector:Conn_01x04_Pin")
-		(at 21.59 53.34 0)
+		(at 21.59 55.88 0)
+		(mirror x)
 		(unit 1)
 		(exclude_from_sim no)
@@
 		(dnp no)
 		(property "Reference" "J2"
-			(at 20.32 55.8801 0)
+			(at 20.32 53.3399 0)
 			(effects
 				(font
@@
 		)
 		(property "Value" "Conn_01x04_Pin"
-			(at 20.32 53.3401 0)
+			(at 20.32 55.8799 0)
 			(effects
 				(font
@@
 		)
 		(property "Footprint" "LCSC:CONN-SMD_HCZZ0451-4"
-			(at 21.59 53.34 0)
+			(at 21.59 55.88 0)
 			(effects
 				(font
@@
 		)
 		(property "Datasheet" "~"
-			(at 21.59 53.34 0)
+			(at 21.59 55.88 0)
 			(effects
 				(font
@@
 		)
 		(property "Description" "Generic connector, single row, 01x04, script generated"
-			(at 21.59 53.34 0)
+			(at 21.59 55.88 0)
 			(effects
 				(font
@@
 		(in_bom yes)
 		(on_board yes)
-		(dnp no)
+		(dnp yes)
 		(property "Reference" "R14"
 			(at 195.072 38.608 90)
