File: Hardware/Powermeter1P1I.kicad_pcb (KiCad board)
At the start: 4 copper layers, 50 x 62 mm, 79 parts, among them IC1 CH32V003F4U6, IC3 RY8310, J1 Conn_01x04_Pin, J2 Conn_01x04_Pin, J3 Conn_01x02_Socket, J4 Conn_01x01_Socket, J5 Conn_01x01_Socket, J6 Conn_01x01_Socket, J7 Conn_01x01_Socket, J8 Conn_01x02_Socket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

Commit message: isolation slot and silkscreen tweaks
Changed lines of the file:
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@@
 			(effects
 				(font
-					(size 1 1)
-					(thickness 0.15)
+					(size 0.6 0.6)
+					(thickness 0.1)
 				)
 			)
@@
 			(at -4.9022 -4.1951 0)
 			(layer "F.SilkS")
+			(hide yes)
 			(effects
 				(font
-					(size 1 1)
-					(thickness 0.15)
+					(size 0.6 0.6)
+					(thickness 0.1)
 				)
 			)
@@
 			(at 0 -5.3 0)
 			(layer "F.SilkS")
+			(hide yes)
 			(effects
 				(font
-					(size 1 1)
-					(thickness 0.15)
+					(size 0.6 0.6)
+					(thickness 0.1)
 				)
 			)
@@
 		(at 138.4078 102.2658 180)
 		(property "Reference" "U4"
-			(at 1.5 -0.5 180)
+			(at 20.0578 13.1158 0)
 			(unlocked yes)
 			(layer "F.SilkS")
 			(effects
 				(font
-					(size 1 1)
-					(thickness 0.15)
+					(size 0.6 0.6)
+					(thickness 0.1)
 				)
 			)
@@
 		(tags "test point THT pad rectangle square")
 		(property "Reference" "J4"
-			(at 0 -2.398 0)
+			(at 0.0858 2.3488 0)
 			(layer "F.SilkS")
 			(effects
 				(font
-					(size 1 1)
-					(thickness 0.15)
+					(size 0.6 0.6)
+					(thickness 0.1)
 				)
 			)
@@
 			(at 0 -5.3 0)
 			(layer "F.SilkS")
+			(hide yes)
 			(effects
 				(font
-					(size 1 1)
-					(thickness 0.15)
+					(size 0.6 0.6)
+					(thickness 0.1)
 				)
 			)
@@
 			(at 0 -5.3 0)
 			(layer "F.SilkS")
+			(hide yes)
 			(effects
 				(font
-					(size 1 1)
-					(thickness 0.15)
+					(size 0.6 0.6)
+					(thickness 0.1)
 				)
 			)
@@
 			(effects
 				(font
-					(size 1 1)
-					(thickness 0.15)
+					(size 0.6 0.6)
+					(thickness 0.1)
 				)
 			)
@@
 			(effects
 				(font
-					(size 1 1)
-					(thickness 0.15)
+					(size 0.6 0.6)
+					(thickness 0.1)
 				)
 			)
@@
 			(effects
 				(font
-					(size 1 1)
-					(thickness 0.15)
+					(size 0.6 0.6)
+					(thickness 0.1)
 				)
 			)
@@
 			(effects
 				(font
-					(size 1 1)
-					(thickness 0.15)
+					(size 0.6 0.6)
+					(thickness 0.1)
 				)
 			)
@@
 			(at 0 2.7 90)
 			(layer "F.SilkS")
+			(hide yes)
 			(effects
 				(font
-					(size 1 1)
-					(thickness 0.15)
+					(size 0.6 0.6)
+					(thickness 0.1)
 				)
 			)
@@
 		(tags "DCDC-Converter TRACO TEA1 THT SIP-4 1W")
 		(property "Reference" "U5"
-			(at 1.6 -3.23 0)
+			(at 6.5568 9.0468 0)
 			(layer "F.SilkS")
 			(effects
 				(font
-					(size 1 1)
-					(thickness 0.15)
+					(size 0.6 0.6)
+					(thickness 0.1)
 				)
 			)
@@
 		(tags "resistor")
 		(property "Reference" "R11"
-			(at 0 1.17 90)
+			(at -0.9108 0.94765 90)
 			(layer "B.SilkS")
 			(effects
@@
 		(tags "resistor")
 		(property "Reference" "R27"
-			(at 0 1.17 0)
+			(at -0.0268 -0.9558 0)
 			(layer "B.SilkS")
 			(effects
 				(font
-					(size 1 1)
-					(thickness 0.15)
+					(size 0.6 0.6)
+					(thickness 0.1)
 				)
 				(justify mirror)
@@
 		(tags "capacitor")
 		(property "Reference" "C2"
-			(at 0 1.16 0)
+			(at -1.421 0.0184 0)
 			(layer "B.SilkS")
 			(effects
@@
 		(tags "capacitor")
 		(property "Reference" "C14"
-			(at 0 1.16 90)
+			(at 1.8451 -0.00235 90)
 			(layer "B.SilkS")
 			(effects
@@
 		(tags "SOT TO_SOT_SMD")
 		(property "Reference" "IC3"
-			(at 0 2.4 0)
+			(at -1.38345 -2.452 0)
 			(layer "B.SilkS")
 			(effects
@@
 		(tags "capacitor")
 		(property "Reference" "C6"
-			(at 0.01305 2.1146 0)
+			(at 3.25025 0.023 0)
 			(layer "B.SilkS")
 			(effects
@@
 		(tags "capacitor")
 		(property "Reference" "C4"
-			(at 0 1.16 90)
+			(at 0.5878 -0.9616 90)
 			(layer "B.SilkS")
 			(effects
@@
 		(tags "resistor")
 		(property "Reference" "R25"
-			(at -1.9012 0.0286 180)
+			(at 1.9692 -0.0202 0)
 			(layer "B.SilkS")
 			(effects
@@
 		(at 161.979 98.803 90)
 		(property "Reference" "D5"
-			(at -2.239 -0.0032 180)
+			(at -2.247 0.371 180)
 			(layer "B.SilkS")
 			(effects
@@
 		(tags "SOD-323")
 		(property "Reference" "D2"
-			(at -0.0984 1.317 0)
+			(at 0.7742 1.317 0)
 			(layer "B.SilkS")
 			(effects
@@
 		(tags "resistor")
 		(property "Reference" "R3"
-			(at 0 1.17 0)
+			(at -1.647 -0.0184 0)
 			(layer "B.SilkS")
 			(effects
@@
 		(tags "diode")
 		(property "Reference" "D4"
-			(at 0 1.17 90)
+			(at 0 -1.288 90)
 			(layer "B.SilkS")
 			(effects
@@
 			(effects
 				(font
-					(size 1 1)
-					(thickness 0.15)
+					(size 0.6 0.6)
+					(thickness 0.1)
 				)
 				(justify mirror)
@@
 		(tags "resistor")
 		(property "Reference" "R2"
-			(at 0 1.17 0)
+			(at -1.7368 -0.0204 0)
 			(layer "B.SilkS")
 			(effects
@@
 		(tags "resistor")
 		(property "Reference" "R17"
-			(at 0 1.17 0)
+			(at -0.0132 -0.9634 0)
 			(layer "B.SilkS")
 			(effects
 				(font
-					(size 1 1)
-					(thickness 0.15)
+					(size 0.6 0.6)
+					(thickness 0.1)
 				)
 				(justify mirror)
@@
 		(tags "resistor")
 		(property "Reference" "R6"
-			(at 0 1.82 90)
+			(at 2.9629 0.021 90)
 			(layer "B.SilkS")
 			(effects
@@
 		(tags "resistor")
 		(property "Reference" "R10"
-			(at 0 1.82 90)
+			(at 3.2512 -0.016 90)
 			(layer "B.SilkS")
 			(effects
@@
 		(tags "resistor")
 		(property "Reference" "R12"
-			(at 0 1.17 90)
+			(at -0.8034 -0.85235 90)
 			(layer "B.SilkS")
 			(effects
@@
 		(at 161.984053 94.6404 90)
 		(property "Reference" "D6"
-			(at 2.5138 0.245747 90)
+			(at 2.2404 0.465947 180)
 			(layer "B.SilkS")
 			(effects
@@
 		(tags "capacitor")
 		(property "Reference" "C1"
-			(at 0 1.16 90)
+			(at 0.0098 -1.0672 90)
 			(layer "B.SilkS")
 			(effects
@@
 		(tags "resistor")
 		(property "Reference" "R1"
-			(at 0 1.17 0)
+			(at -1.5802 0.0086 0)
 			(layer "B.SilkS")
 			(effects
@@
 		(tags "capacitor")
 		(property "Reference" "C19"
-			(at 3.1394 81.2792 90)
+			(at 0 -1.0772 90)
 			(layer "B.SilkS")
 			(effects
 				(font
-					(size 1 1)
-					(thickness 0.15)
+					(size 0.6 0.6)
+					(thickness 0.1)
 				)
 				(justify mirror)
@@
 		(tags "capacitor")
 		(property "Reference" "R5"
-			(at 0 1.16 0)
+			(at 0 -0.8894 0)
 			(layer "B.SilkS")
 			(effects
@@
 		(tags "TSOT-23")
 		(property "Reference" "Q2"
-			(at 0 0 0)
+			(at 1.8836 1.566 0)
 			(layer "B.SilkS")
 			(effects
@@
 		(at 148.5646 78.3336 -90)
 		(property "Reference" "U3"
-			(at 0 4.95 90)
+			(at -1.4336 -1.0854 180)
 			(layer "B.SilkS")
 			(effects
@@
 		(tags "capacitor")
 		(property "Reference" "C5"
-			(at 0 2.3 90)
+			(at -0.0025 1.86555 90)
 			(layer "B.SilkS")
 			(effects
@@
 		(tags "SOIC SO")
 		(property "Reference" "U7"
-			(at 0 6.1 90)
+			(at -2.9808 6.0518 90)
 			(layer "B.SilkS")
 			(effects
@@
 		(tags "capacitor")
 		(property "Reference" "C10"
-			(at 0 1.16 90)
+			(at -0.0306 0.87495 90)
 			(layer "B.SilkS")
 			(effects
@@
 		(at 161.9758 72.8726 90)
 		(property "Reference" "D3"
-			(at 0 4.2 90)
+			(at -2.5774 -0.0258 0)
 			(layer "B.SilkS")
 			(effects
@@
 		(at 149.7584 124.9608)
 		(property "Reference" "SW1"
-			(at 0 4.77 0)
+			(at 0 -1.3108 0)
 			(layer "B.SilkS")
 			(effects
 				(font
-					(size 1 1)
-					(thickness 0.15)
+					(size 0.6 0.6)
+					(thickness 0.1)
 				)
 				(justify mirror)
@@
 		(at 151.3994 72.5047 90)
 		(property "Reference" "U2"
-			(at 3.1373 0.01 180)
+			(at 3.2047 1.8006 180)
 			(layer "B.SilkS")
 			(effects
@@
 		(at 120.73675 90.6095)
 		(property "Reference" "L2"
-			(at 0 4 0)
+			(at 0.01325 -1.5595 0)
 			(layer "B.SilkS")
 			(effects
@@
 		(model "${KIPRJMOD}/LCSC.3dshapes/IND-SMD_L2.0-W1.6-H1.1.wrl"
 			(offset
-				(xyz -4.16 -2.29 -0)
+				(xyz 0 0 -0)
 			)
 			(scale
@@
 			)
 			(rotate
-				(xyz 0 0 270)
+				(xyz 0 0 -90)
 			)
 		)
@@
 		(tags "capacitor")
 		(property "Reference" "C11"
-			(at 0 1.16 0)
+			(at 0 -1.103 0)
 			(layer "B.SilkS")
 			(effects
@@
 	(gr_poly
 		(pts
+			(xy 167.1 87.400075) (xy 167.1 88.8) (xy 133.04286 88.8) (xy 131.5 86.099995) (xy 131.5 83.9) (xy 108.9 83.9)
+			(xy 108.9 83.25) (xy 132.2 83.25) (xy 132.2 85.051779) (xy 133.55 87.349971)
+		)
+		(stroke
+			(width 0)
+			(type solid)
+		)
+		(fill solid)
+		(layer "B.Mask")
+	)
+	(gr_poly
+		(pts
 			(xy 165.595426 72.8218) (xy 165.575905 72.548865) (xy 165.517741 72.281486) (xy 165.422116 72.025106)
 			(xy 165.290978 71.784945) (xy 165.126996 71.565891) (xy 164.933509 71.372404) (xy 164.714455 71.208422)
@@
 		)
 		(stroke
+			(width 0)
+			(type solid)
+		)
+		(fill solid)
+		(layer "F.Mask")
+	)
+	(gr_poly
+		(pts
+			(xy 167.1 87.400075) (xy 167.1 88.8) (xy 133.04286 88.8) (xy 131.5 86.099995) (xy 131.5 83.9) (xy 108.9 83.9)
+			(xy 108.9 83.25) (xy 132.2 83.25) (xy 132.2 85.051779) (xy 133.55 87.349971)
+		)
+		(stroke
