File: Hardware/Powermeter1P1I.kicad_sch (KiCad schematic)
At the start: 12 parts, among them IC1 CH32V003F4U6, J9 TagConnect

Commit message: add all
Parts:
- added R27: 4k7, Resistor_SMD:R_0402_1005Metric, symbol Device:R
- added SW1: SW_Push, LCSC:SW-SMD_TS24CA, symbol Switch:SW_Push
Connections:
- net +5V: now also R27.1
- net GND: now also SW1.1
- net Button: now reaches IC1.5 (PD0)
- net Button: now also R27.2, SW1.2
- no-connect marks 5 -> 4
