File: Hardware/P1I1_PowerMetering.kicad_sch (KiCad schematic)
At the start: 34 parts, among them J10 Conn_01x04_Pin, J3 Conn_01x02_Socket, J4 Conn_01x01_Socket, J5 Conn_01x01_Socket, J6 Conn_01x01_Socket, J7 Conn_01x01_Socket, J8 Conn_01x02_Socket, U2 BL0942_C2909509, U3 XC6206P332MR, U5 TEA1-0505

Commit message: add all
Parts:
- removed J10: Conn_01x04_Pin, LCSC:CONN-SMD_HCZZ0451-4, symbol Connector:Conn_01x04_Pin
Connections:
- net GND1: now also C7.2, R21.2
- net MISO_ISO: now also U2.14 (TX/SDO); no longer U2.13 (RX/SDI)
- net MOSI_ISO: now also U2.13 (RX/SDI); no longer U2.14 (TX/SDO)
- no-connect marks 0 -> 3
Other:
- moved on the sheet: C7, R17, R21, R29

Commit message: isolation slot and silkscreen tweaks
Parts:
- U7: value ~ -> CA-IS3541
Changed lines of the file:
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@@
 		(on_board yes)
 		(dnp no)
-		(fields_autoplaced yes)
 		(property "Reference" "U7"
-			(at 205.3941 87.63 0)
+			(at 207.01 114.046 0)
 			(effects
 				(font
@@
 			)
 		)
-		(property "Value" "~"
-			(at 205.3941 90.17 0)
+		(property "Value" "CA-IS3541"
+			(at 207.01 116.84 0)
 			(effects
 				(font
